File: Hardware/SparkFun_TPL5110_Nano_Power_Switch.brd (EAGLE design)
At the start: 25.4 x 25.4 mm, 62 parts, among them Q1 1.1A/60V/600mΩ, SW1 DIP-06, U1 TPL5110

Commit message: Switches gate and source nets, attaches LED to VDD_OUT, adds "+" and "-" silk to board
Parts:
- R6: value 330 -> 1k
- moved U$4 2.59 mm to (11.4, 1.60)
- moved U$1 2.54 mm to (14.0, 1.68)
- moved U$33 0.57 mm to (11.1, 4.19)
- moved U$34 0.51 mm to (15.8, 4.29)
- moved LOGO2 0.36 mm to (22.9, 19.6), turned to 90 degrees
- turned Q1 to 180 degrees
Connections:
- net DONE: now also J2.3; no longer J2.4
- net GND: now also J2.4; no longer J2.3
- net VDD: now also Q1.2; no longer JP2.2, Q1.3
- net VDD_OUT: now also JP2.2, Q1.3; no longer Q1.2
Routing:
- net VDD_OUT: track 4.97 -> 40.3 mm, vias 0 -> 1
- net VDD: track 54.4 -> 31.6 mm, vias 1 -> 0
- net !DRV: track 9.10 -> 12.7 mm
- net DONE: track 11.3 -> 10.0 mm
Other:
- board text added: "+"
- board text added: "-"
